Commit message: working rviz diff control

File: src/r5_description/description/ros2_control/r5.ros2_control.urdf.xacro (robot description, xacro)
@@ -1,9 +1,9 @@
-<?xml version="1.0" ?>
-<robot xmlns:xacro="http://wiki.ros.org/xacro">
+<?xml version="1.0"?>
+<robot xmlns:xacro="http://www.ros.org/wiki/xacro">
     <xacro:macro name="r5_ros2_control" params="name prefix use_mock_hardware">
         <ros2_control name="${name}" type="system">
             <hardware>
                 <plugin>r5/DiffBotSystemHardware</plugin>
-                <param name="example_paramhw_start_duration_sec">1.0</param>
+                <param name="example_param_hw_start_duration_sec">1.0</param>
                 <param name="example_param_hw_stop_duration_sec">3.0</param>
             </hardware>

File: src/r5_description/description/urdf/mech/wheel.urdf.xacro (robot description, xacro)
@@ -32,6 +32,6 @@
                 <mass value="${wheel_mass}"/>
                 <inertia
-                  ixx="${(wheel_mass/12.0) * (3*wheel_radius*wheel_radius + wheel_width*wheel_width)}" ixy="0" ixz="0"
-                  iyy="${(wheel_mass/2.0) * (wheel_radius*wheel_radius)}" iyz="0"
+                  ixx="${(wheel_mass/12.0) * (3*wheel_radius*wheel_radius + wheel_width*wheel_width)}" ixy="0.0" ixz="0.0"
+                  iyy="${(wheel_mass/2.0) * (wheel_radius*wheel_radius)}" iyz="0.0"
                   izz="${(wheel_mass/12.0) * (3*wheel_radius*wheel_radius + wheel_width*wheel_width)}"/>
               </inertial>
@@ -42,5 +42,6 @@
             <child link="${prefix}${side}_wheel"/>
             <axis xyz="0 1 0"/>
-            <limit effort="50.0" velocity="10.0"/>
+            <limit effort="50.0" velocity="3.0"/>
+            <dynamics damping="0.2"/>
         </joint>
         <transmission name="${prefix}${side}_wheel_trans" type="SimpleTransmission">

File: src/r5_description/description/urdf/r5.urdf.xacro (robot description, xacro)
@@ -7,8 +7,10 @@
   <xacro:arg name="prefix" default=""/>
   <xacro:arg name="use_gazebo" default="false"/>
+  <xacro:arg name="use_mock_hardware" default="false" />
   <xacro:include filename="$(find r5)/urdf/sensors/lidar.urdf.xacro" />
   <xacro:include filename="$(find r5)/urdf/sensors/imu.urdf.xacro"/>
   <xacro:include filename="$(find r5)/urdf/mech/wheel.urdf.xacro"/>
   <xacro:include filename="$(find r5)/urdf/mech/r5_base.urdf.xacro"/>
+  <xacro:include filename="$(find r5)/ros2_control/r5.ros2_control.urdf.xacro" />
   <xacro:r5_base prefix="$(arg prefix)"/>
   <!-- Front Right (FR) -->
@@ -65,10 +67,5 @@
     update_rate="15.0"
     topic_name="imu/data"/>
-  <!-- <xacro:include filename="$(find r5)/urdf/control/diff_drive_control_plugin.urdf.xacro" />
-  <xacro:load_diff_drive_control_plugin use_gazebo="$(arg use_gazebo)"/> -->
-  <!-- <xacro:include filename="$(find r5)/urdf/control/velocity_control_plugin.urdf.xacro" />
-  <xacro:load_velocity_control_plugin use_gazebo="$(arg use_gazebo)"/> -->
-  <xacro:include filename="$(find r5)/ros2_control/r5.ros2_control.urdf.xacro" />
   <xacro:r5_ros2_control
-    prefix="$(arg prefix)" name="DiffBot" use_mock_hardware="$(arg use_mock_hardware)"/>
+    name="$(arg robot_name)" prefix="$(arg prefix)"  use_mock_hardware="$(arg use_mock_hardware)"/>
 </robot>
